Commit message: 8-dof controller

File: uibk_robot_driver/model/robotinoarm.urdf (robot description, URDF)
Before this commit: robot robotinoarm, 8 links, 7 joints
Links:
- link link1: geometry collision mesh filename=package://uibk_robot_driver/model/meshes/link1_collision.stl; visual mesh filename=package://uibk_robot_driver/model/meshes/link1.stl
- link link2: geometry collision mesh filename=package://uibk_robot_driver/model/meshes/link2_collision.stl; visual mesh filename=package://uibk_robot_driver/model/meshes/link2.stl
- link link3: geometry collision mesh filename=package://uibk_robot_driver/model/meshes/link3_collision.stl; visual mesh filename=package://uibk_robot_driver/model/meshes/link3.stl
- link link4: geometry collision mesh filename=package://uibk_robot_driver/model/meshes/link4_collision.stl; visual mesh filename=package://uibk_robot_driver/model/meshes/link4.stl
- link linkbasemotor: geometry collision mesh filename=package://uibk_robot_driver/model/meshes/motor1_collision.s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; visual mesh filename=package://uibk_robot_driver/model/meshes/motor1.stl
